File: EL6170_Pro_Max_Plus.kicad_sch (KiCad schematic)
At the start: 87 parts, among them CN1 PJ-327A0-SMT, J1 USB_C_Receptacle, J2 microSD, Q1 MMBT3904, Q2 MMBT3904, SW1 RST, SW2 BOOT, U1 ESP32-S3, U10 ME6211C33M5, U11 IP5306, U2 TPS61040DBV, U3 ESP-PSRAM64H, U4 W25Q128JVS, U5 ME6217C33M5, U6 CH340K, U7 RFANT5220110A0T, U8 CH334R, U9 PCM5102A, X1 40MHz, X2 12MHz

Commit message: sync
Parts:
- removed U11: IP5306, easyeda2kicad:ESOP-8_L4.9-W3.9-P1.27-LS6.0-BL-EP, symbol easyeda2kicad:IP5306
Changed lines of the file:
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@@
-	)
-	(symbol
-		(lib_id "easyeda2kicad:IP5306")
-		(at 46.99 213.36 0)
-		(unit 1)
-		(exclude_from_sim no)
-		(in_bom yes)
-		(on_board yes)
-		(dnp no)
-		(fields_autoplaced yes)
-		(property "Reference" "U11"
-			(at 46.99 226.06 0)
-			(effects
-				(font
-					(size 1.27 1.27)
-				)
-			)
-		)
-		(property "Value" "IP5306"
-			(at 46.99 228.6 0)
-			(effects
-				(font
-					(size 1.27 1.27)
-				)
-			)
-		)
-		(property "Footprint" "easyeda2kicad:ESOP-8_L4.9-W3.9-P1.27-LS6.0-BL-EP"
-			(at 46.99 228.6 0)
-			(effects
-				(font
-					(size 1.27 1.27)
-				)
-				(hide yes)
-			)
-		)
-		(property "Datasheet" "https://lcsc.com/product-detail/PMIC-Battery-Management_IP5306_C181692.html"
-			(at 46.99 231.14 0)
-			(effects
-				(font
-					(size 1.27 1.27)
-				)
-				(hide yes)
-			)
-		)
-		(property "Description" ""
-			(at 46.99 213.36 0)
-			(effects
-				(font
-					(size 1.27 1.27)
-				)
-				(hide yes)
-			)
-		)
-		(property "LCSC Part" "C181692"
-			(at 46.99 233.68 0)
-			(effects
-				(font
-					(size 1.27 1.27)
-				)
-				(hide yes)
-			)
-		)
-		(pin "1"
-		)
-		(pin "3"
-		)
-		(pin "7"
-		)
-		(pin "8"
-		)
-		(pin "2"
-		)
-		(pin "5"
-		)
-		(pin "6"
-		)
-		(pin "9"
-		)
-		(pin "4"
-		)
-		(instances
-			(project ""
-				(path "/b3287cc9-c0c8-4939-96d8-31efd376f189"
-					(reference "U11")
-					(unit 1)
-				)
-			)
-		)
 	)
 	(symbol

Commit message: sync
Connections:
- net +3V3: no longer C36.1, U10.1 (V_{IN}), U10.3 (CE)
- net +5V: now also C36.1, U10.1 (V_{IN}), U10.3 (CE)
Changed lines of the file:
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@@
-	)
-	(symbol
-		(lib_id "power:+3V3")
-		(at 254 175.26 0)
-		(unit 1)
-		(exclude_from_sim no)
-		(in_bom yes)
-		(on_board yes)
-		(dnp no)
-		(fields_autoplaced yes)
-		(property "Reference" "#PWR071"
-			(at 254 179.07 0)
-			(effects
-				(font
-					(size 1.27 1.27)
-				)
-				(hide yes)
-			)
-		)
-		(property "Value" "+3V3"
-			(at 254 170.18 0)
-			(effects
-				(font
-					(size 1.27 1.27)
-				)
-			)
-		)
-		(property "Footprint" ""
-			(at 254 175.26 0)
-			(effects
-				(font
-					(size 1.27 1.27)
-				)
-				(hide yes)
-			)
-		)
-		(property "Datasheet" ""
-			(at 254 175.26 0)
-			(effects
-				(font
-					(size 1.27 1.27)
-				)
-				(hide yes)
-			)
-		)
-		(property "Description" "Power symbol creates a global label with name \"+3V3\""
-			(at 254 175.26 0)
-			(effects
-				(font
-					(size 1.27 1.27)
-				)
-				(hide yes)
-			)
-		)
-		(pin "1"
-		)
-		(instances
-			(project "EL6170_Pro_Max_Plus"
-				(path "/b3287cc9-c0c8-4939-96d8-31efd376f189"
-					(reference "#PWR071")
-					(unit 1)
-				)
-			)
-		)
 	)
 	(symbol
@@
 					(unit 1)
 				)
+			)
+		)
+	)
+	(symbol
+		(lib_id "power:+5V")
+		(at 254 175.26 0)
+		(unit 1)
+		(exclude_from_sim no)
+		(in_bom yes)
+		(on_board yes)
+		(dnp no)
+		(fields_autoplaced yes)
+		(property "Reference" "#PWR071"
+			(at 254 179.07 0)
+			(effects
+				(font
+					(size 1.27 1.27)
+				)
+				(hide yes)
+			)
+		)
+		(property "Value" "+5V"
+			(at 254 170.18 0)
+			(effects
+				(font
+					(size 1.27 1.27)
+				)
+			)
+		)
+		(property "Footprint" ""
+			(at 254 175.26 0)
+			(effects
+				(font
+					(size 1.27 1.27)
+				)
+				(hide yes)
+			)
+		)
+		(property "Datasheet" ""
+			(at 254 175.26 0)
+			(effects
+				(font
+					(size 1.27 1.27)
+				)
+				(hide yes)
+			)
+		)
+		(property "Description" "Power symbol creates a global label with name \"+5V\""
+			(at 254 175.26 0)
+			(effects
+				(font
+					(size 1.27 1.27)
+				)
+				(hide yes)
+			)
+		)
+		(pin "1"
+		)
+		(instances
+			(project "EL6170_Pro_Max_Plus"
+				(path "/b3287cc9-c0c8-4939-96d8-31efd376f189"
+					(reference "#PWR071")
+					(unit 1)
+				)

Commit message: power mang
Parts:
- added C38, C42: 0.1uF, SparkFun-Capacitor:C_0603_1608Metric, symbol SparkFun-Capacitor:0.1uF_0603_25V_20%
- added C39: 47uF, SparkFun-Capacitor:C_0805_2012Metric, symbol SparkFun-Capacitor:47uF_0805_6.3V_20%
- added C40, C41: 22uF, SparkFun-Capacitor:C_0603_1608Metric, symbol SparkFun-Capacitor:22uF_0603_6.3V_20%
- added C43: 10uF, SparkFun-Capacitor:C_0603_1608Metric, symbol SparkFun-Capacitor:10uF_0603_10V_20%
- added D5: SS34, Diode_SMD:D_SMA, symbol Diode:SS34
- added L6: SCCD43-220KT, easyeda2kicad:IND-SMD_L4.5-W4.0_SCCD43, symbol easyeda2kicad:SCCD43-220KT
- added Q3: 2N7002, Package_TO_SOT_SMD:SOT-23, symbol Transistor_FET:2N7002
- added Q4, Q5: AO3401A, Package_TO_SOT_SMD:SOT-23, symbol Transistor_FET:AO3401A
- added R21, R22: 330, SparkFun-Resistor:R_0603_1608Metric, symbol SparkFun-Resistor:330_0603
- added R23: 2, SparkFun-Resistor:R_0603_1608Metric, symbol SparkFun-Resistor:2.2k_0603
- added U11: TP5400_C2891434, easyeda2kicad:ESOP-8_L4.9-W3.9-P1.27-LS6.0-BL-EP, symbol easyeda2kicad:TP5400_C2891434
Connections:
- net +5V: now also Q4.2 (S), Q5.2 (S), R22.1; no longer J1.VBUS
- net GND: now also C38.2, C39.2, C40.2, C41.2, C42.2, C43.2, Q3.2 (S), R21.2, R23.2, U11.7 (GND), U11.9 (EP)
- new net: Q3.3 (D), Q5.1 (G), R22.2
- new net: R23.1, U11.3 (PROG)
- new net: D5.2 (A), L6.1, U11.8 (LX)
- new net BAT5V: C38.1, C39.1, D5.1 (K), Q3.1 (G), Q4.1 (G), Q5.3 (D), R21.1, U11.1 (VOUT)
- new net CHRG: U11.2 (~{CHRG})
- new net STDBY: U11.4 (~{STDBY})
- new net USB5V: C43.1, J1.VBUS, Q4.3 (D), U11.5 (VCC)
- new net VBAT: C40.1, C41.1, C42.1, L6.2, U11.6 (BAT)
