File: EL6170_Pro_Max_Plus.kicad_pcb (KiCad board)
At the start: 4 copper layers, 128 x 70.5 mm, 233 parts, among them CN1 PJ-327A0-SMT, J1 USB_C_Receptacle, J2 microSD, Q1 MMBT3904, Q2 MMBT3904, Q3 2N7002, Q4 AO3401A, Q5 AO3401A, SW1 SW_LEFT, SW10 SW_K4, SW11 SW_K5, SW12 SW_K6, SW13 SW_K7, SW14 SW_K8, SW15 SW_K9, SW16 SW_K0, SW17 SW_KQ, SW18 SW_KW, SW19 SW_KE, SW2 SW_UP, SW20 SW_KR, SW21 SW_KT, SW22 SW_KY, SW23 SW_KU, SW24 SW_KI, SW25 SW_KO, SW26 SW_KP, SW27 SW_KA, SW28 SW_KS, SW29 SW_KD, SW3 SW_DOWN, SW30 SW_KF, SW31 SW_KG, SW32 SW_KH, SW33 SW_KJ, SW34 SW_KK, SW35 SW_KL, SW36 SW_KZ, SW37 SW_KX, SW38 SW_KC, SW39 SW_KV, SW4 SW_RIGHT, SW40 SW_KB, SW41 SW_KN, SW42 SW_KM, SW43 SW_KCOM, SW44 SW_KDOT, SW45 SW_SHIFT, SW46 SW_CE(IO0), SW47 SW_OFF, SW48 SW_SECRET, SW49 SW_MCK, SW5 SW_UP2, SW50 SW_SPACE, SW51 SW_REMARK, SW52 SW_CALENDAR, SW53 SW_MODE, SW54 SW_ENTER, SW6 SW_DOWN2, SW7 SW_K1, SW8 SW_K2, SW9 SW_K3, U1 ESP32-S3, U10 ME6211C33M5, U11 TP5400_C2891434, U12 PCF8575DBR, U2 TPS61040DBV, U3 ESP-PSRAM64H, U4 W25Q128JVS, U5 ME6217C33M5, U6 CH340K, U7 RFANT5220110A0T, U8 CH334R, U9 PCM5102A, X1 40MHz, X2 12MHz

Commit message: sync
Parts:
- moved C18 1.00 mm to (106.0, 127.0)
- moved C45 0.98 mm to (103.5, 127.0)
- moved U7 0.60 mm to (151.9, 130.8)
- moved C10 0.51 mm to (95.9, 129.0)
- moved C19 0.50 mm to (100.7, 131.3)
- moved C9 0.50 mm to (95.9, 125.9)
- moved C13 0.22 mm to (97.4, 130.9)
- moved C44 0.20 mm to (106.0, 130.9)
- moved C25 0.18 mm to (103.5, 130.9)
Routing:
- net KEY_COL6: track 0.00 -> 175.6 mm, vias 0 -> 8
- net KEY_COL7: track 0.00 -> 162.5 mm, vias 0 -> 13
- net KEY_ROW0: track 0.00 -> 152.9 mm, vias 0 -> 5
- net KEY_ROW2: track 0.00 -> 133.8 mm, vias 0 -> 7
- net KEY_ROW3: track 0.00 -> 129.1 mm, vias 0 -> 11
- net KEY_ROW4: track 0.00 -> 127.9 mm, vias 0 -> 8
- net KEY_ROW1: track 0.00 -> 104.5 mm, vias 0 -> 2
- net Net-(D47-A): track 0.00 -> 100.2 mm, vias 0 -> 9
- net Net-(D56-A): track 0.00 -> 99.2 mm, vias 0 -> 4
- net Net-(D64-A): track 0.00 -> 94.6 mm, vias 0 -> 5
- net Net-(D63-A): track 0.00 -> 87.0 mm, vias 0 -> 6
- net KEY_ROW5: track 0.00 -> 78.1 mm, vias 0 -> 6
- net Net-(D57-A): track 0.00 -> 76.1 mm, vias 0 -> 2
- net Net-(D62-A): track 0.00 -> 71.5 mm, vias 0 -> 4
- net Net-(D58-A): track 0.00 -> 69.8 mm, vias 0 -> 2
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
Commit message: sync
Routing:
- net Net-(D13-A): track 0.00 -> 34.1 mm, vias 0 -> 1
- net Net-(D34-A): track 0.00 -> 29.1 mm, vias 0 -> 2
- net Net-(D35-A): track 0.00 -> 27.9 mm, vias 0 -> 3
- net Net-(D27-A): track 0.00 -> 22.1 mm, vias 0 -> 3
- net Net-(D44-A): track 0.00 -> 19.3 mm, vias 0 -> 1
- net Net-(D26-A): track 0.00 -> 16.9 mm, vias 0 -> 3
- net Net-(D25-A): track 0.00 -> 13.9 mm, vias 0 -> 2
- net Net-(D14-A): track 0.00 -> 12.7 mm, vias 0 -> 1
- net Net-(D36-A): track 0.00 -> 12.4 mm, vias 0 -> 2
- net Net-(D24-A): track 0.00 -> 10.5 mm, vias 0 -> 2
- net Net-(D16-A): track 0.00 -> 7.56 mm, vias 0 -> 1
- net Net-(D28-A): track 0.00 -> 2.14 mm, vias 0 -> 1
- net +3V3: track 374.8 -> 374.0 mm
- net XOUT: track 13.1 -> 13.7 mm
- net DEMP: vias 0 -> 68
- added copper zone on In1.Cu, net DEMP
- added copper zone on In2.Cu, net DEMP
